File: non-nemo/non_nemo.kicad_pcb (KiCad board)
At the start: 2 copper layers, 260.1 x 100.6 mm, 92 parts, among them J1 Conn_BAT, J2 Conn_BAT, X1 5.5mm, X10 5.5mm, X2 5.5mm, X3 5.5mm, X4 5.5mm, X5 5.5mm, X6 5.5mm, X7 5.5mm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

Commit message: artwork
Parts:
- moved D19 15.0 mm to (259.8, 97.0), turned to -90 degrees
- moved D20 15.0 mm to (259.8, 78.0), turned to -90 degrees
- moved D21 15.0 mm to (259.8, 59.0), turned to -90 degrees
- moved D22 15.0 mm to (240.8, 97.0), turned to -90 degrees
- moved D23 15.0 mm to (240.8, 78.0), turned to -90 degrees
- moved D24 15.0 mm to (240.8, 59.0), turned to -90 degrees
- moved D25 15.0 mm to (221.8, 97.0), turned to -90 degrees
- moved D26 15.0 mm to (221.8, 78.0), turned to -90 degrees
- moved D27 15.0 mm to (221.8, 59.0), turned to -90 degrees
- moved D28 15.0 mm to (202.8, 97.0), turned to -90 degrees
- moved D29 15.0 mm to (202.8, 78.0), turned to -90 degrees
- moved D30 15.0 mm to (202.8, 59.0), turned to -90 degrees
- moved D31 15.0 mm to (183.8, 97.0), turned to -90 degrees
- moved D32 15.0 mm to (183.8, 78.0), turned to -90 degrees
- moved D33 15.0 mm to (183.8, 59.0), turned to -90 degrees
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Routing:
- net col_pinky_r: track 0.00 -> 194.6 mm, vias 0 -> 1
- net col_middle: track 0.00 -> 179.0 mm
- net col_middle_r: track 0.00 -> 177.4 mm
- net col_pinky: track 0.00 -> 169.5 mm
- net col_ring_r: track 0.00 -> 165.8 mm, vias 0 -> 1
- net col_index: track 0.00 -> 157.9 mm
- net col_index_r: track 0.00 -> 151.1 mm
- net col_ring: track 0.00 -> 150.6 mm
- net row_top_r: track 0.00 -> 150.3 mm, vias 0 -> 1
- net row_top: track 0.00 -> 131.9 mm
- net row_home_r: track 0.00 -> 128.7 mm, vias 0 -> 1
- net row_bottom: track 0.00 -> 127.9 mm
- net col_inner_r: track 0.00 -> 127.6 mm
- net row_home: track 0.00 -> 116.5 mm
- net col_inner: track 0.00 -> 114.4 mm
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