File: non-nemo-low/non_nemo.kicad_pcb (KiCad board)
At the start: 2 copper layers, 260.1 x 100.6 mm, 92 parts, among them J1 Conn_BAT, J2 Conn_BAT, X1 5.5mm, X10 5.5mm, X2 5.5mm, X3 5.5mm, X4 5.5mm, X5 5.5mm, X6 5.5mm, X7 5.5mm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

Commit message: small tweaks
Routing:
- net col_ring_r: track 165.8 -> 166.5 mm
- net col_pinky_r: track 194.6 -> 195.3 mm
Other:
- board text added: "Low Profile"
- board text added: "Non Nemo 3x5 Split Ergo Mechanican Keyboard"
