File: non-nemo-low/non_nemo_low.kicad_pcb (KiCad board)
At the start: 2 copper layers, 260.1 x 100.6 mm, 92 parts, among them J1 Conn_BAT, J2 Conn_BAT, X1 5.5mm, X10 5.5mm, X2 5.5mm, X3 5.5mm, X4 5.5mm, X5 5.5mm, X6 5.5mm, X7 5.5mm, X8 5.5mm, X9 5.5mm

Commit message: Low Profile
pogopin and reset button
Parts:
- added J3: Conn_BAT, TB2086_MISC:Molex_Pico-EZmate_78171-0002_1x02-1MP_P1.20mm_HandSolder, F.Cu at (130.7, 105.5)
- added J4: Conn_BAT, TB2086_MISC:Molex_Pico-EZmate_78171-0002_1x02-1MP_P1.20mm_HandSolder, F.Cu at (166.6, 105.5)
- added RSW1: SMT 2X4X3.5MM Tactile Tact Push Button, TB2086_SMD:SMT 2X4X3.5MM Tactile Tact Push Button, F.Cu at (144.7, 95.0)
- added RSW2: SMT 2X4X3.5MM Tactile Tact Push Button, TB2086_SMD:SMT 2X4X3.5MM Tactile Tact Push Button, F.Cu at (152.6, 95.0)
- J1, J2: value Conn_BAT -> Conn_01x02; footprint TB2086_MISC:Molex_Pico-EZmate_78171-0002_1x02-1MP_P1.20mm_HandSolder -> TB2086_MISC:Tag_Pogopin_1x02_P2.54mm
- moved X7 161.3 mm to (267.3, 45.7)
- moved X5 160.8 mm to (30.0, 45.7), turned to 90 degrees
- moved X9 85.2 mm to (151.4, 121.0), turned to 0 degrees
- moved X6 76.0 mm to (106.0, 45.7)
- moved X8 76.0 mm to (191.3, 45.7)
- moved X3 66.3 mm to (200.8, 136.3)
- moved X1 57.0 mm to (96.5, 136.3), turned to -90 degrees
- moved X2 38.0 mm to (134.5, 136.3)
- moved X4 38.0 mm to (162.8, 136.3)
- moved J1 12.8 mm to (141.5, 98.6), turned to 90 degrees
- moved J2 12.8 mm to (155.8, 98.6)
- moved SW_SPDT1 0.20 mm to (143.5, 105.5)
- moved SW_SPDT2 0.20 mm to (153.8, 105.5)
Connections:
- J1 pad 1: GND -> BAT
- J1 pad 2: Net-(J1-Pin_2) -> RST
- J2 pad 1: GND -> BAT_r
- J2 pad 2: Net-(J2-Pin_2) -> RST_r
- SW_SPDT1 pad : (no net) -> GND
- SW_SPDT1 pad 2: Net-(J1-Pin_2) -> Net-(J3-Pin_2)
- SW_SPDT2 pad : (no net) -> GND
- SW_SPDT2 pad 2: Net-(J2-Pin_2) -> Net-(J4-Pin_2)
Routing:
- net Net-(J3-Pin_2): track 0.00 -> 9.81 mm
- net Net-(J1-Pin_2): track 9.81 -> 0.00 mm
- net Net-(J2-Pin_2): track 9.81 -> 0.00 mm
- net Net-(J4-Pin_2): track 0.00 -> 9.81 mm
- net BAT_r: track 0.00 -> 3.62 mm
- net BAT: track 0.00 -> 3.62 mm
- net row_bottom: track 127.9 -> 124.6 mm
- net RST: track 0.00 -> 2.13 mm
- net RST_r: track 0.00 -> 2.13 mm
- net col_ring_r: track 166.5 -> 164.9 mm
- net col_pinky_r: track 195.3 -> 193.7 mm
- net row_thumb_r: track 66.1 -> 66.8 mm
- net row_thumb: track 79.8 -> 79.1 mm
- net GND: vias 0 -> 2
Other:
- board text added: "B+"
- board text added: "Non Nemo 0.2.0"
- board text added: "RST"
- board text removed: "Non Nemo 0.1.6"

Commit message: fixed footprint layer for low
Parts:
- D1, D10, D11, D12, D13, D14, D15, D16, D17, D18, D19, D2, D20, D21, D22, D23, D24, D25, D26, D27, D28, D29, D3, D30, D31, D32, D33, D34, D35, D36, D4, D5, D6, D7, D8, D9: value D -> 1N4148W; footprint TB2086_SMD:TB2086_SMD_D3_SMD -> TB2086_SMD:D3_SMD; moved to B.Cu
- J1, J2, J3, J4, LOGO2, LOGO4, MCU1, MCU2, RSW1, RSW2, S1, S10, S11, S12, S13, S14, S15, S16, S17, S18, S19, S2, S20, S21, S22, S23, S24, S25, S26, S27, S28, S29, S3, S30, S31, S32, S33, S34, S35, S36, S4, S5, S6, S7, S8, S9, SW_SPDT1, SW_SPDT2, X7: moved to B.Cu
