File: non-nemo-low/non_nemo_low.kicad_sch (KiCad schematic)
At the start: 82 parts, among them J1 Conn_BAT, J2 Conn_BAT

Commit message: reset switch (#6)
* added reset switch

* Low Profile

pogopin and reset button

* MX Profile

pogopin and reset switch

* MX Profile PCB

* Chimera

pogopin and reset switch

* version

* updated README.md
Parts:
- added J1, J2: Conn_01x02, TB2086_MISC:Tag_Pogopin_1x02_P2.54mm, symbol Connector_Generic:Conn_01x02
- added RSW1, RSW2: SMT 2X4X3.5MM Tactile Tact Push Button, TB2086_SMD:SMT 2X4X3.5MM Tactile Tact Push Button, symbol TB2086_SMD:SMT 2X4X3.5MM Tactile Tact Push Button
- renumbered J1 to J3, J2 to J4
Connections:
- net BAT: now also J1.1 (Pin_1)
- net BAT_r: now also J2.1 (Pin_1)
- net GND: now also RSW1.2, RSW2.1
- new net RST: J1.2 (Pin_2), RSW1.1
- new net RST_r: J2.2 (Pin_2), RSW2.2
Other:
- title: (none) -> Non Nemo Low Profile
- moved on the sheet: J3, J4

Commit message: fixed footprint layer for low
Parts:
- D1, D10, D11, D12, D13, D14, D15, D16, D17, D18, D19, D2, D20, D21, D22, D23, D24, D25, D26, D27, D28, D29, D3, D30, D31, D32, D33, D34, D35, D36, D4, D5, D6, D7, D8, D9: value D -> 1N4148W
Changed lines of the file:
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@@
 			)
 		)
-		(property "Value" "D"
+		(property "Value" "1N4148W"
 			(at 136.652 55.372 0)
 			(effects
@@
 					(size 1.27 1.27)
 				)
+				    (hide yes)
 			)
 		)
@@
 			)
 		)
-		(property "Value" "D"
+		(property "Value" "1N4148W"
 			(at 329.438 170.688 0)
 			(effects
@@
 					(size 1.27 1.27)
 				)
+				    (hide yes)
 			)
 		)
@@
 			)
 		)
-		(property "Value" "D"
+		(property "Value" "1N4148W"
 			(at 293.878 170.688 0)
 			(effects
@@
 					(size 1.27 1.27)
 				)
+				    (hide yes)
 			)
 		)
@@
 			)
 		)
-		(property "Value" "D"
+		(property "Value" "1N4148W"
 			(at 118.872 76.454 0)
 			(effects
@@
 					(size 1.27 1.27)
 				)
+				    (hide yes)
 			)
 		)
@@
 			)
 		)
-		(property "Value" "D"
+		(property "Value" "1N4148W"
 			(at 329.438 210.82 0)
 			(effects
@@
 					(size 1.27 1.27)
 				)
+				    (hide yes)
 			)
 		)
@@
 			)
 		)
-		(property "Value" "D"
+		(property "Value" "1N4148W"
 			(at 118.872 55.372 0)
 			(effects
@@
 					(size 1.27 1.27)
 				)
+				    (hide yes)
 			)
 		)
@@
 			)
 		)
-		(property "Value" "D"
+		(property "Value" "1N4148W"
 			(at 364.998 230.632 0)
 			(effects
@@
 					(size 1.27 1.27)
 				)
+				    (hide yes)
 			)
 		)
@@
 			)
 		)
-		(property "Value" "D"
+		(property "Value" "1N4148W"
 			(at 118.872 95.504 0)
 			(effects
@@
 					(size 1.27 1.27)
 				)
+				    (hide yes)
 			)
 		)
@@
 			)
 		)
-		(property "Value" "D"
+		(property "Value" "1N4148W"
 			(at 347.218 170.688 0)
 			(effects
@@
 					(size 1.27 1.27)
 				)
+				    (hide yes)
 			)
 		)
@@
 			)
 		)
-		(property "Value" "D"
+		(property "Value" "1N4148W"
 			(at 364.998 170.688 0)
 			(effects
@@
 					(size 1.27 1.27)
 				)
+				    (hide yes)
 			)
 		)
@@
 			)
 		)
-		(property "Value" "D"
+		(property "Value" "1N4148W"
 			(at 172.212 55.372 0)
 			(effects
@@
 					(size 1.27 1.27)
 				)
+				    (hide yes)
 			)
 		)
@@
 			)
 		)
-		(property "Value" "D"
+		(property "Value" "1N4148W"
 			(at 154.432 95.504 0)
 			(effects
@@
 					(size 1.27 1.27)
 				)
+				    (hide yes)
 			)
 		)
@@
 			)
 		)
-		(property "Value" "D"
+		(property "Value" "1N4148W"
 			(at 311.658 210.82 0)
 			(effects
@@
 					(size 1.27 1.27)
 				)
+				    (hide yes)
 			)
 		)
@@
 			)
 		)
-		(property "Value" "D"
+		(property "Value" "1N4148W"
 			(at 136.652 95.504 0)
 			(effects
@@
 					(size 1.27 1.27)
 				)
+				    (hide yes)
 			)
 		)
@@
 			)
 		)
-		(property "Value" "D"
+		(property "Value" "1N4148W"
 			(at 101.092 55.372 0)
 			(effects
@@
 					(size 1.27 1.27)
 				)
+				    (hide yes)
 			)
 		)
@@
 			)
 		)
-		(property "Value" "D"
+		(property "Value" "1N4148W"
 			(at 172.212 115.316 0)
 			(effects
@@
 					(size 1.27 1.27)
 				)
+				    (hide yes)
 			)
 		)
@@
 			)
 		)
-		(property "Value" "D"
+		(property "Value" "1N4148W"
 			(at 347.218 191.77 0)
 			(effects
@@
 					(size 1.27 1.27)
 				)
+				    (hide yes)
 			)
 		)
@@
 			)
 		)
-		(property "Value" "D"
+		(property "Value" "1N4148W"
 			(at 154.432 55.372 0)
 			(effects
@@
 					(size 1.27 1.27)
 				)
+				    (hide yes)
 			)
 		)
@@
 			)
 		)
-		(property "Value" "D"
+		(property "Value" "1N4148W"
 			(at 329.438 230.632 0)
 			(effects
@@
 					(size 1.27 1.27)
 				)
+				    (hide yes)
 			)
 		)
@@
 			)
 		)
-		(property "Value" "D"
+		(property "Value" "1N4148W"
 			(at 364.998 191.77 0)
 			(effects
@@
 					(size 1.27 1.27)
 				)
+				    (hide yes)
 			)
 		)
@@
 			)
 		)
-		(property "Value" "D"
+		(property "Value" "1N4148W"
 			(at 154.432 76.454 0)
 			(effects
@@
 					(size 1.27 1.27)
 				)
+				    (hide yes)
 			)
 		)
@@
 			)
 		)
-		(property "Value" "D"
+		(property "Value" "1N4148W"
 			(at 154.432 115.316 0)
 			(effects
@@
 					(size 1.27 1.27)
 				)
+				    (hide yes)
 			)
 		)
@@
 			)
 		)
-		(property "Value" "D"
+		(property "Value" "1N4148W"
 			(at 136.652 76.454 0)
 			(effects
@@
 					(size 1.27 1.27)
 				)
+				    (hide yes)
 			)
 		)
@@
 			)
 		)
-		(property "Value" "D"
+		(property "Value" "1N4148W"
 			(at 172.212 76.454 0)
 			(effects
@@
 					(size 1.27 1.27)
 				)
+				    (hide yes)
 			)
 		)
@@
 			)
 		)
-		(property "Value" "D"
+		(property "Value" "1N4148W"
 			(at 364.998 210.82 0)
 			(effects
@@
 					(size 1.27 1.27)
 				)
+				    (hide yes)
 			)
 		)
@@
 			)
 		)
-		(property "Value" "D"
+		(property "Value" "1N4148W"
 			(at 172.212 95.504 0)
 			(effects
@@
 					(size 1.27 1.27)
 				)
+				    (hide yes)
 			)
 		)
@@
 			)
 		)
-		(property "Value" "D"
+		(property "Value" "1N4148W"
 			(at 101.092 76.454 0)
 			(effects
@@
 					(size 1.27 1.27)
 				)
+				    (hide yes)
 			)
 		)
@@
 			)
 		)
-		(property "Value" "D"
+		(property "Value" "1N4148W"
 			(at 293.878 210.82 0)
 			(effects
@@
 					(size 1.27 1.27)
 				)
+				    (hide yes)
 			)
 		)
@@
 			)
 		)
-		(property "Value" "D"
+		(property "Value" "1N4148W"
 			(at 347.218 210.82 0)
 			(effects
@@
 					(size 1.27 1.27)
 				)
+				(hide yes)
 			)
 		)
@@
 			)
 		)
-		(property "Value" "D"
+		(property "Value" "1N4148W"
 			(at 136.652 115.316 0)
 			(effects
@@
 			)
 		)
-		(property "Value" "D"
+		(property "Value" "1N4148W"
 			(at 329.438 191.77 0)
 			(effects
@@
 			)
 		)
-		(property "Value" "D"
+		(property "Value" "1N4148W"
 			(at 347.218 230.632 0)
 			(effects
@@
 			)
 		)
-		(property "Value" "D"
+		(property "Value" "1N4148W"
 			(at 311.658 170.688 0)
 			(effects
@@
 			)
 		)
-		(property "Value" "D"
+		(property "Value" "1N4148W"
 			(at 293.878 191.77 0)
 			(effects
@@
 			)
 		)
-		(property "Value" "D"
+		(property "Value" "1N4148W"
 			(at 311.658 191.77 0)
 			(effects
@@
 			)
 		)
-		(property "Value" "D"
+		(property "Value" "1N4148W"
 			(at 101.092 95.504 0)
 			(effects
