File: plates/low-profile/bottom.kicad_pcb (KiCad board)
At the start: 2 copper layers, 260.1 x 100.6 mm, 12 parts, among them X1 5.5mm, X10 5.5mm, X2 5.5mm, X3 5.5mm, X4 5.5mm, X5 5.5mm, X6 5.5mm, X7 5.5mm, X8 5.5mm, X9 5.5mm

Commit message: small tweaks
Other:
- board text added: "Low Profile"
- board text added: "Non Nemo 3x5 Split Ergo Mechanican Keyboard"
