File: plates/low-profile/bottom_low.kicad_pcb (KiCad board)
At the start: 2 copper layers, 260.1 x 100.6 mm, 12 parts, among them X1 5.5mm, X10 5.5mm, X2 5.5mm, X3 5.5mm, X4 5.5mm, X5 5.5mm, X6 5.5mm, X7 5.5mm, X8 5.5mm, X9 5.5mm

Commit message: Low Profile
pogopin and reset button
Parts:
- added J1: Conn_01x02, TB2086_MISC:Pogopin_1x02_P2.54mm, F.Cu at (135.1, 85.1)
- added J2: Conn_01x02, TB2086_MISC:Pogopin_1x02_P2.54mm, F.Cu at (171.0, 85.1)
- added J3: Conn_01x02, TB2086_MISC:Pogopin_1x02_P2.54mm, F.Cu at (130.7, 80.4)
- added J4: Conn_01x02, TB2086_MISC:Pogopin_1x02_P2.54mm, F.Cu at (166.6, 80.4)
- added J5: Conn_01x02, TB2086_MISC:Pogopin_1x02_P2.54mm, F.Cu at (141.5, 98.6)
- added J6: Conn_01x02, TB2086_MISC:Pogopin_1x02_P2.54mm, F.Cu at (155.8, 98.6)
- added JP1: SolderJumper_3_Open, TB2086_MISC:SolderJumper-3_P1.3mm_Open_RoundedPad1.0x1.5mm, F.Cu at (130.7, 89.8)
- added JP2: SolderJumper_3_Open, TB2086_MISC:SolderJumper-3_P1.3mm_Open_RoundedPad1.0x1.5mm, F.Cu at (166.6, 89.8)
- moved X7 161.3 mm to (267.3, 45.7)
- moved X5 160.8 mm to (30.0, 45.7), turned to 90 degrees
- moved X9 85.2 mm to (151.4, 121.0), turned to 0 degrees
- moved X6 76.0 mm to (106.0, 45.7)
- moved X8 76.0 mm to (191.3, 45.7)
- moved X3 66.3 mm to (200.8, 136.3)
- moved X1 57.0 mm to (96.5, 136.3), turned to -90 degrees
- moved X2 38.0 mm to (134.5, 136.3)
- moved X4 38.0 mm to (162.8, 136.3)
Routing:
- net RST_r: track 0.00 -> 25.8 mm
- net RST: track 0.00 -> 24.7 mm
- net BAT: track 0.00 -> 20.3 mm
- net BAT_r: track 0.00 -> 20.2 mm
- net BAT_c: track 0.00 -> 9.89 mm
- net BAT_cr: track 0.00 -> 9.86 mm
- net BAT_xr: track 0.00 -> 5.58 mm
- net BAT_x: track 0.00 -> 5.54 mm
Other:
- board text added: "B+"
- board text added: "GND"
- board text added: "MINI"
- board text added: "RST"
- board text added: "XIAO"
