File: plates/low-profile/top_low.kicad_pcb (KiCad board)
At the start: 2 copper layers, 260.1 x 100.6 mm, 9 parts, among them X1 5.5mm, X2 5.5mm, X3 5.5mm, X4 5.5mm, X5 5.5mm, X6 5.5mm, X7 5.5mm, X8 5.5mm, X9 5.5mm

Commit message: Low Profile
pogopin and reset button
Other:
- board text added: "Non Nemo 0.2.0"
- board text removed: "Non Nemo 0.1.6"
Changed lines of the file:
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@@
 	(title_block
 		(title "top")
-		(date "2025-04-06")
-		(rev "0.1.6")
+		(date "2025-04-09")
+		(rev "0.2.0")
 		(company "Allen Choi")
 	)
@@
 		(layer "Edge.Cuts")
 	)
-	(gr_text "Non Nemo 0.1.6"
+	(gr_text "Non Nemo 0.2.0"
 		(at 49 109.5 0)
 		(layer "B.SilkS")
@@
 		)
 	)
-	(gr_text "Non Nemo 0.1.6"
+	(gr_text "Non Nemo 0.2.0"
 		(at 248.3 109.5 0)
 		(layer "B.SilkS")
