File: non-nemo-chimera/non_nemo_chimera.kicad_sch (KiCad schematic)
At the start: 82 parts, among them J1 Conn_BAT, J2 Conn_BAT

Commit message: reset switch (#6)
* added reset switch

* Low Profile

pogopin and reset button

* MX Profile

pogopin and reset switch

* MX Profile PCB

* Chimera

pogopin and reset switch

* version

* updated README.md
Parts:
- removed J1, J2: Conn_BAT, TB2086_SMD:Molex_Pico-EZmate_78171-0002_1x02-1MP_P1.20mm_HandSolder, symbol Connector_Generic_MountingPin:Conn_01x02_MountingPin
- added J1, J2: Conn_01x02, TB2086_MISC:Tag_Pogopin_1x02_P2.54mm, symbol Connector_Generic:Conn_01x02
- added J3, J4: Conn_BAT, TB2086_SMD:Molex_Pico-EZmate_78171-0002_1x02-1MP_P1.20mm_HandSolder, symbol Connector_Generic_MountingPin:Conn_01x02_MountingPin
- added RSW1, RSW2: SMT 2X4X3.5MM Tactile Tact Push Button, TB2086_SMD:SMT 2X4X3.5MM Tactile Tact Push Button, symbol TB2086_SMD:SMT 2X4X3.5MM Tactile Tact Push Button
- renumbered D19 to D16, D20 to D17, D21 to D18, D22 to D19, D23 to D20, D24 to D21, D25 to D22, D26 to D23, D27 to D24, D28 to D25, D29 to D26, D30 to D27, D31 to D28, D32 to D29, D33 to D30, D16 to D31, D17 to D32, D18 to D33, S19 to S16, S20 to S17, S21 to S18, S22 to S19, S23 to S20, S24 to S21, S25 to S22, S26 to S23, S27 to S24, S28 to S25, S29 to S26, S30 to S27, S31 to S28, S32 to S29, S33 to S30, S16 to S31, S17 to S32, S18 to S33
Connections:
- net BAT: now also J1.1 (Pin_1)
- net BAT_r: now also J2.1 (Pin_1)
- net GND: now also J3.1 (Pin_1), J3.MP (MountPin), J4.1 (Pin_1), J4.MP (MountPin), RSW1.2, RSW2.1
- net at SW_SPDT2.2 (B): now also J4.2 (Pin_2)
- net at SW_SPDT1.2 (B): now also J3.2 (Pin_2)
- new net RST: J1.2 (Pin_2), RSW1.1
- new net RST_r: J2.2 (Pin_2), RSW2.2
Other:
- title: (none) -> Non Nemo Chimera
