File: non-nemo-mx/non_nemo_mx.kicad_pcb (KiCad board)
At the start: 2 copper layers, 273.7 x 107 mm, 92 parts, among them J1 Conn_BAT, J2 Conn_BAT, X1 5.5mm, X10 5.5mm, X2 5.5mm, X3 5.5mm, X4 5.5mm, X5 5.5mm, X6 5.5mm, X7 5.5mm, X8 5.5mm, X9 5.5mm

Commit message: reset switch (#6)
* added reset switch

* Low Profile

pogopin and reset button

* MX Profile

pogopin and reset switch

* MX Profile PCB

* Chimera

pogopin and reset switch

* version

* updated README.md
Parts:
- added J3: Conn_BAT, TB2086_MISC:Molex_Pico-EZmate_78171-0002_1x02-1MP_P1.20mm_HandSolder, F.Cu at (136.0, 104.5)
- added J4: Conn_BAT, TB2086_MISC:Molex_Pico-EZmate_78171-0002_1x02-1MP_P1.20mm_HandSolder, F.Cu at (173.5, 104.5)
- added RSW1: SMT 2X4X3.5MM Tactile Tact Push Button, TB2086_SMD:SMT 2X4X3.5MM Tactile Tact Push Button, F.Cu at (150.8, 94.0)
- added RSW2: SMT 2X4X3.5MM Tactile Tact Push Button, TB2086_SMD:SMT 2X4X3.5MM Tactile Tact Push Button, F.Cu at (158.7, 94.0)
- J1, J2: value Conn_BAT -> Conn_01x02; footprint TB2086_MISC:Molex_Pico-EZmate_78171-0002_1x02-1MP_P1.20mm_HandSolder -> TB2086_MISC:Tag_Pogopin_1x02_P2.54mm
- moved X5 169.9 mm to (30.0, 42.5), turned to 90 degrees
- moved X7 169.5 mm to (279.5, 42.5)
- moved X9 88.1 mm to (157.5, 120.0), turned to 0 degrees
- moved X6 80.0 mm to (110.0, 42.5)
- moved X8 80.0 mm to (199.5, 42.5)
- moved X3 69.5 mm to (209.5, 139.5)
- moved X1 60.7 mm to (100.0, 139.5), turned to -90 degrees
- moved X2 40.0 mm to (140.0, 139.5)
- moved X4 40.0 mm to (169.5, 139.5)
- moved J1 13.5 mm to (147.6, 97.6), turned to 90 degrees
- moved J2 13.5 mm to (161.9, 97.6)
Connections:
- J1 pad 1: GND -> BAT
- J1 pad 2: Net-(J1-Pin_2) -> RST
- J2 pad 1: GND -> BAT_r
- J2 pad 2: Net-(J2-Pin_2) -> RST_r
- SW_SPDT1 pad : (no net) -> GND
- SW_SPDT1 pad 2: Net-(J1-Pin_2) -> Net-(J3-Pin_2)
- SW_SPDT2 pad : (no net) -> GND
- SW_SPDT2 pad 2: Net-(J2-Pin_2) -> Net-(J4-Pin_2)
Routing:
- net Net-(J4-Pin_2): track 0.00 -> 10.8 mm
- net Net-(J2-Pin_2): track 10.8 -> 0.00 mm
- net Net-(J3-Pin_2): track 0.00 -> 10.8 mm
- net Net-(J1-Pin_2): track 10.8 -> 0.00 mm
- net col_index_r: track 163.1 -> 158.7 mm, vias 0 -> 1
- net col_middle_r: track 188.0 -> 183.7 mm, vias 0 -> 1
- net col_ring_r: track 164.4 -> 160.4 mm, vias 0 -> 1
- net col_pinky_r: track 185.6 -> 181.7 mm, vias 0 -> 1
- net BAT_r: track 0.00 -> 3.62 mm
- net BAT: track 0.00 -> 3.62 mm
- net RST: track 0.00 -> 2.30 mm
- net RST_r: track 0.00 -> 2.27 mm
- net col_inner_r: track 152.1 -> 149.9 mm
- net row_thumb_r: track 104.2 -> 104.8 mm
Other:
- board text added: "B+"
- board text added: "Non Nemo 0.2.0"
- board text added: "RST"
- board text removed: "Non Nemo 0.1.6"

Commit message: fixed footprint layer for mx
Parts:
- D1, D10, D11, D12, D13, D14, D15, D16, D17, D18, D19, D2, D20, D21, D22, D23, D24, D25, D26, D27, D28, D29, D3, D30, D31, D32, D33, D34, D35, D36, D4, D5, D6, D7, D8, D9: value D -> 1N4148W; footprint TB2086_SMD:TB2086_SMD_D3_SMD -> TB2086_SMD:D3_SMD; moved to B.Cu
- J1, J2, J3, J4, LOGO2, LOGO4, MCU1, MCU2, RSW1, RSW2, S1, S10, S11, S12, S13, S14, S15, S16, S17, S18, S19, S2, S20, S21, S22, S23, S24, S25, S26, S27, S28, S29, S3, S30, S31, S32, S33, S34, S35, S36, S4, S5, S6, S7, S8, S9, SW_SPDT1, SW_SPDT2: moved to B.Cu
