File: wired/non-nemo-chimera/non_nemo_chimera_wired.kicad_sch (KiCad schematic)
At the start: 84 parts

Commit message: Chimera Wired + Case (#10)
* Updated cases for Chimera Wired

* updated README.md for Chimera Wired

* updated github workflow
Other:
- title: Non Nemo Chimera -> Non Nemo Chimera Wired
Changed lines of the file:
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@@
 	(paper "A3")
 	(title_block
-		(title "Non Nemo Chimera")
-		(date "2025-04-09")
-		(rev "0.2.0")
+		(title "Non Nemo Chimera Wired")
+		(date "2025-04-21")
+		(rev "0.2.1")
 	)
 	(junction
