File: wireless/non-nemo-chimera/non_nemo_chimera.kicad_pcb (KiCad board)
At the start: 2 copper layers, 273.7 x 107 mm, 96 parts, among them J1 Conn_01x02, J2 Conn_01x02, J3 Conn_BAT, J4 Conn_BAT, X1 5.5mm, X10 5.5mm, X2 5.5mm, X3 5.5mm, X4 5.5mm, X5 5.5mm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

Commit message: added standoff holes for case
Non Nemo Chimera Wireless
Routing:
- net row_bottom_r: track 131.0 -> 154.2 mm
- net row_home_r: track 222.1 -> 230.7 mm
- net col_pinky_r: track 182.0 -> 186.9 mm
- net col_inner: track 169.0 -> 172.5 mm
- net col_inner_r: track 152.0 -> 148.7 mm
- net col_index_r: track 161.4 -> 164.3 mm
- net col_index: track 191.2 -> 188.8 mm
- net col_middle: track 209.2 -> 211.0 mm
- net col_ring: track 158.1 -> 159.9 mm
- net col_middle_r: track 186.8 -> 187.6 mm
- net row_top_r: track 187.7 -> 188.4 mm
Other:
- outline, holes or cut-outs redrawn

Commit message: updated README.md
Other:
- board text added: "Non Nemo 0.2.1"
- board text removed: "Non Nemo 0.2.0"
Changed lines of the file:
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@@
 		)
 	)
-	(gr_text "Non Nemo 0.2.0"
+	(gr_text "Non Nemo 0.2.1"
 		(at 259.5 109.5 0)
 		(layer "B.SilkS")
@@
 		)
 	)
-	(gr_text "Non Nemo 0.2.0"
+	(gr_text "Non Nemo 0.2.1"
 		(at 50 109.5 0)
 		(layer "B.SilkS")
