File: wireless/non-nemo-mx/non_nemo_mx.kicad_pcb (KiCad board)
At the start: 2 copper layers, 273.7 x 107 mm, 96 parts, among them J1 Conn_01x02, J2 Conn_01x02, J3 Conn_BAT, J4 Conn_BAT, X1 5.5mm, X10 5.5mm, X2 5.5mm, X3 5.5mm, X4 5.5mm, X5 5.5mm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

Commit message: fixed Wired (#12)
* fixed Non Nemo Wired

* fixed ergogen for Wired
Routing:
- net row_thumb_r: track 104.8 -> 125.1 mm
- net row_thumb: track 105.7 -> 125.6 mm
- net col_pinky_r: track 181.7 -> 191.6 mm
- net row_home_r: track 221.9 -> 229.6 mm
- net col_index_r: track 158.7 -> 163.3 mm
- net col_middle_r: track 183.7 -> 186.1 mm
- net col_ring_r: track 160.4 -> 158.8 mm
- net col_ring: track 158.1 -> 159.2 mm
- net col_middle: track 188.7 -> 189.8 mm
- net col_inner_r: track 149.9 -> 150.6 mm
Other:
- outline, holes or cut-outs redrawn
- board text added: "Non Nemo 0.2.1"
- board text removed: "Non Nemo 0.2.0"
